File: pcb/TashRecorder.kicad_pcb (KiCad board)
At the start: 4 copper layers, 56.6 x 57.7 mm, 53 parts, among them J1 RCJ-013, J2 Mini-DIN-8, J3 Conn_01x04, SW1 EG 1224 SPDT, U1 LM385Z-2.5, U2 LM385Z-2.5, U3 OPA2337, U4 PIC12F1501-xP

Commit message: minot schematic fixes (typos), 3D render fixes for PCB
Parts:
- R14, R15: value 47 -> 47Ω
- R7: value 220k -> 220kΩ
