File: pcb/TashRecorder.kicad_sch (KiCad schematic)
At the start: 49 parts, among them J1 RCJ-013, J2 Mini-DIN-8, J3 Conn_01x04, SW1 EG 1224 SPDT, U1 LM385Z-2.5, U2 LM385Z-2.5, U3 OPA2337, U4 PIC12F1501-xP

Commit message: minot schematic fixes (typos), 3D render fixes for PCB
Parts:
- J3: now not fitted
Changed lines of the file:
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@@
 	(title_block
 		(title "TashRecorder")
-		(date "2024-06-02")
+		(date "2024-10-06")
 		(rev "2.1")
 		(company "Lostwave")
@@
 		(at 166.37 106.68 0)
 		(unit 1)
-		(exclude_from_sim no)
+		(exclude_from_sim yes)
 		(in_bom no)
 		(on_board yes)
-		(dnp no)
+		(dnp yes)
 		(fields_autoplaced yes)
 		(property "Reference" "J3"
